File: SHT-3x-hat.kicad_pcb (KiCad board)
At the start: 2 copper layers, 4 parts, among them J1 Power, U1 ESP-01, U2 SHT31, U3 AMS1117-3.3

Commit message: added edge cuts
Other:
- board outline added: 26.7 x 19.1 mm
Changed lines of the file:
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@@
   (general
     (thickness 1.6)
-    (drawings 0)
+    (drawings 6)
     (tracks 29)
     (zones 0)
@@
     )
   )
+  (gr_line (start 107.95 120.65) (end 109.22 120.65) (layer Edge.Cuts) (width 0.05))
+  (gr_line (start 107.95 101.6) (end 107.95 120.65) (layer Edge.Cuts) (width 0.05))
+  (gr_line (start 109.22 101.6) (end 107.95 101.6) (layer Edge.Cuts) (width 0.05))
+  (gr_line (start 134.62 101.6) (end 109.22 101.6) (layer Edge.Cuts) (width 0.05))
+  (gr_line (start 134.62 120.65) (end 134.62 101.6) (layer Edge.Cuts) (width 0.05))
+  (gr_line (start 109.22 120.65) (end 134.62 120.65) (layer Edge.Cuts) (width 0.05))
   (segment (start 114.3 107.998686) (end 114.3 109.22) (width 1) (layer F.Cu) (net 1))
   (segment (start 114.3 107.882081) (end 114.3 107.998686) (width 1) (layer F.Cu) (net 1))
